Commit message: added angular limits

File: pinc_open_driver/urdf/gripper_macros.xacro (robot description, xacro)
@@ -17,5 +17,5 @@
     <origin xyz="0.053492 0 0.0"/>
     <axis xyz="0 0 1"/>
-    <limit lower="-2.44" upper="0" effort="5" velocity="1"/>
+    <limit lower="-2.653" upper="0.1745" effort="5" velocity="1"/>
   </joint>
   <joint name="${prefix}base_link_to_right_arm" type="revolute">

File: pinc_open_driver/urdf/gripper_ros2_control.xacro (robot description, xacro)
@@ -33,6 +33,6 @@
     <joint name="${prefix}gripper">
       <command_interface name="position">
-        <param name="min">-2.44</param>
-        <param name="max">0.0</param>
+        <param name="min">-2.653</param>
+        <param name="max">0.1745</param>
       </command_interface>
       <xacro:if value="${use_mock_hardware}">
@@ -56,4 +56,7 @@
         <param name="ID">${dxl_id}</param>
         <param name="Operating Mode">${operating_mode}</param>  <!-- 3 = position, 5 = current-based position -->
+        <!-- Servo position limits in raw ticks (2048 = 0 rad), 3 deg beyond the software limits -->
+        <param name="Min Position Limit">285</param>
+        <param name="Max Position Limit">2196</param>
         <command_interface name="Goal Position"/>
         <state_interface name="Present Position"/>
